File: board/mcu_reset.kicad_sch (KiCad schematic)
At the start: 4 parts, among them SW501 RST

Commit message: finish board design
Changed lines of the file:
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@@
   (symbol (lib_id "Device:R") (at 64.77 55.88 90) (unit 1)
     (in_bom yes) (on_board yes) (dnp no) (fields_autoplaced)
-    (property "Reference" "R502" (at 64.77 50.8 90)
+    (property "Reference" "R502" (at 64.77 49.53 90)
       (effects (font (size 1.27 1.27)))
     )
-    (property "Value" "330Ω" (at 64.77 53.34 90)
+    (property "Value" "330Ω" (at 64.77 52.07 90)
       (effects (font (size 1.27 1.27)))
     )
@@
       (project "eprom5vread"
         (path "/b08a8275-42d3-43c1-b04c-f89506e7527b/2fd5d481-fecc-449f-aabd-88adee8fd543/6327e597-74ae-4074-90f5-37ad20c0474e"
-          (reference "R3") (unit 1)
+          (reference "R102") (unit 1)
         )
       )
@@
   (symbol (lib_id "Switch:SW_Push") (at 73.66 62.23 90) (unit 1)
     (in_bom yes) (on_board yes) (dnp no) (fields_autoplaced)
-    (property "Reference" "SW501" (at 74.93 61.595 90)
+    (property "Reference" "SW501" (at 74.93 60.96 90)
       (effects (font (size 1.27 1.27)) (justify right))
     )
-    (property "Value" "RST" (at 74.93 64.135 90)
+    (property "Value" "RST" (at 74.93 63.5 90)
       (effects (font (size 1.27 1.27)) (justify right))
     )
@@
       (project "eprom5vread"
         (path "/b08a8275-42d3-43c1-b04c-f89506e7527b/2fd5d481-fecc-449f-aabd-88adee8fd543/6327e597-74ae-4074-90f5-37ad20c0474e"
-          (reference "SW1") (unit 1)
+          (reference "SW101") (unit 1)
         )
       )
@@
   (symbol (lib_id "Device:C") (at 57.15 62.23 180) (unit 1)
     (in_bom yes) (on_board yes) (dnp no) (fields_autoplaced)
-    (property "Reference" "C501" (at 60.96 61.595 0)
+    (property "Reference" "C501" (at 60.96 60.96 0)
       (effects (font (size 1.27 1.27)) (justify right))
     )
-    (property "Value" "100nF" (at 60.96 64.135 0)
+    (property "Value" "100nF" (at 60.96 63.5 0)
       (effects (font (size 1.27 1.27)) (justify right))
     )
@@
       (project "eprom5vread"
         (path "/b08a8275-42d3-43c1-b04c-f89506e7527b/2fd5d481-fecc-449f-aabd-88adee8fd543/6327e597-74ae-4074-90f5-37ad20c0474e"
-          (reference "C21") (unit 1)
+          (reference "C105") (unit 1)
         )
       )
@@
   (symbol (lib_id "Device:R") (at 48.26 49.53 180) (unit 1)
     (in_bom yes) (on_board yes) (dnp no) (fields_autoplaced)
-    (property "Reference" "R501" (at 50.8 48.895 0)
+    (property "Reference" "R501" (at 50.8 48.26 0)
       (effects (font (size 1.27 1.27)) (justify right))
     )
-    (property "Value" "2.2kΩ" (at 50.8 51.435 0)
+    (property "Value" "2.2kΩ" (at 50.8 50.8 0)
       (effects (font (size 1.27 1.27)) (justify right))
     )
@@
       (project "eprom5vread"
         (path "/b08a8275-42d3-43c1-b04c-f89506e7527b/2fd5d481-fecc-449f-aabd-88adee8fd543/6327e597-74ae-4074-90f5-37ad20c0474e"
-          (reference "R2") (unit 1)
+          (reference "R101") (unit 1)
         )
       )
