File: board/mcu_debug.kicad_sch (KiCad schematic)
At the start: 1 part, among them J4 DEBUG

Commit message: finish board design
Parts:
- renumbered J4 to J101
Changed lines of the file:
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@@
   (symbol (lib_id "Connector_Generic:Conn_02x05_Odd_Even") (at 63.5 62.23 0) (unit 1)
     (in_bom yes) (on_board yes) (dnp no) (fields_autoplaced)
-    (property "Reference" "J4" (at 64.77 50.8 0)
+    (property "Reference" "J101" (at 64.77 50.8 0)
       (effects (font (size 1.27 1.27)))
     )
@@
       (project "eprom5vread"
         (path "/b08a8275-42d3-43c1-b04c-f89506e7527b/2fd5d481-fecc-449f-aabd-88adee8fd543/39033807-b906-459f-a233-a45afe12edb8"
-          (reference "J4") (unit 1)
+          (reference "J101") (unit 1)
         )
       )

Commit message: allow driving ~RESET pins of I2C I/O expanders, add missing resistors
Parts:
- J101: LCSC (none) -> C5250218
Changed lines of the file:
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@@
+			)
+		)
+		(property "LCSC" "C5250218"
+			(at 63.5 62.23 0)
+			(effects
+				(font
+					(size 1.27 1.27)
+				)
+				(hide yes)
 			)
 		)
